File: examples/f35_ducted_quad/electronics/rl_fc_f405/rl_fc_f405.kicad_pcb (KiCad board)
At the start: 4 copper layers, 36 x 36 mm, 65 parts, among them J1 BATT, J2 USB-C, J3 ESC, J4 RX, J5 VTX, J6 SWD, SW1 BOOT, U1 TPS5430, U2 AP2112K-3.3, U3 STM32F405RGT6, U4 ICM-20602, U5 BMP280, U6 W25Q128JV, U7 USBLC6-2SC6, Y1 8MHz

Commit message: Power-stage rework, current-aware review
Parts:
- C5: moved to B.Cu
- moved C5 20.3 mm to (114.6, 127.4), turned to 90 degrees
- moved C2 9.09 mm to (104.0, 124.5), turned to 180 degrees
- moved R2 9.02 mm to (102.6, 116.0), turned to 180 degrees
- moved C1 7.94 mm to (105.3, 124.5), turned to 180 degrees
- moved C3 7.72 mm to (109.8, 119.5), turned to -90 degrees
- moved R1 7.50 mm to (102.6, 117.4), turned to 0 degrees
- moved L1 1.15 mm to (112.2, 127.0)
- turned U1 to -90 degrees
Routing:
- net VBAT: track 65.0 -> 24.2 mm, vias 1 -> 2
- net /Power/BUCK_SW: track 22.1 -> 0.00 mm
- net GND: track 88.5 -> 80.2 mm, vias 34 -> 35
- net /Power/BUCK_FB: track 5.74 -> 2.88 mm
- net +5V: track 94.2 -> 96.4 mm, vias 4 -> 10
- net VBAT_SENSE: track 40.7 -> 41.5 mm
- added copper zone on F.Cu, net /Power/BUCK_SW
- added copper zone on F.Cu, net GND
